File: MRLY220519.kicad_pcb (KiCad board)
At the start: 2 copper layers, 9 parts, among them K1 OMRON G6H-2-100, K2 OMRON G6H-2-100, P1 Terminal Block 8 3.81 Straight

Commit message: update
Parts:
- moved R3 26.8 mm to (149.1, 84.8)
- moved P1 16.6 mm to (127.0, 85.1), turned to 90 degrees
Changed lines of the file:
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@@
   )
   (footprint "Connectors:Terminal Block 1x08 P3.81 Straight" (layer "F.Cu")
-    (at 143.51 86.868 -90)
+    (at 127 85.09 90)
     (property "Comment" "MRT9P3.81/8")
     (property "Manufacturer" "Stelvio")
@@
     (fp_line (start 16.129 -4.826) (end -16.129 -4.826) (layer "F.CrtYd") (width 0.05))
     (fp_line (start 16.129 -4.826) (end 16.129 2.794) (layer "F.CrtYd") (width 0.05))
-    (pad "1" thru_hole rect (at -13.335 0) (size 2 2) (drill 1.2) (layers *.Cu *.Mask)
+    (pad "1" thru_hole rect (at -13.335 0 180) (size 2 2) (drill 1.2) (layers *.Cu *.Mask)
       (net 7 "GND") (pinfunction "Pin_a1") (pintype "passive"))
-    (pad "2" thru_hole oval (at -9.525 0) (size 2 2) (drill 1.2) (layers *.Cu *.Mask)
+    (pad "2" thru_hole oval (at -9.525 0 180) (size 2 2) (drill 1.2) (layers *.Cu *.Mask)
       (net 1 "/+24V") (pintype "passive"))
-    (pad "3" thru_hole oval (at -5.715 0) (size 2 2) (drill 1.2) (layers *.Cu *.Mask)
+    (pad "3" thru_hole oval (at -5.715 0 180) (size 2 2) (drill 1.2) (layers *.Cu *.Mask)
       (net 16 "unconnected-(P1-Pad3)") (pintype "passive+no_connect"))
-    (pad "4" thru_hole oval (at -1.905 0) (size 2 2) (drill 1.2) (layers *.Cu *.Mask)
+    (pad "4" thru_hole oval (at -1.905 0 180) (size 2 2) (drill 1.2) (layers *.Cu *.Mask)
       (net 12 "/K1a") (pintype "passive"))
-    (pad "5" thru_hole oval (at 1.905 0) (size 2 2) (drill 1.2) (layers *.Cu *.Mask)
+    (pad "5" thru_hole oval (at 1.905 0 180) (size 2 2) (drill 1.2) (layers *.Cu *.Mask)
       (net 13 "/K1b") (pintype "passive"))
-    (pad "6" thru_hole oval (at 5.715 0) (size 2 2) (drill 1.2) (layers *.Cu *.Mask)
+    (pad "6" thru_hole oval (at 5.715 0 180) (size 2 2) (drill 1.2) (layers *.Cu *.Mask)
       (net 14 "/K2a") (pintype "passive"))
-    (pad "7" thru_hole oval (at 9.525 0) (size 2 2) (drill 1.2) (layers *.Cu *.Mask)
+    (pad "7" thru_hole oval (at 9.525 0 180) (size 2 2) (drill 1.2) (layers *.Cu *.Mask)
       (net 15 "/K2b") (pintype "passive"))
-    (pad "8" thru_hole oval (at 13.335 0) (size 2 2) (drill 1.2) (layers *.Cu *.Mask)
+    (pad "8" thru_hole oval (at 13.335 0 180) (size 2 2) (drill 1.2) (layers *.Cu *.Mask)
       (net 3 "/+12V") (pintype "passive"))
     (model "${KNV_MODELS}/Terminal Block 8 3.81 Straight.STEP"
@@
   )
   (footprint "Passive:R0207 Axial Horizontal" (layer "F.Cu")
-    (at 166.878 64.77 180)
+    (at 149.098 84.836 180)
     (property "Comment" "1K00")
     (property "Manufacturer" "LSE")

Commit message: update
Parts:
- P1: footprint Connectors:Terminal Block 1x08 P3.81 Straight -> Connectors:Terminal Block 01x08 P3.81 Horizontal
- moved P1 13.1 mm to (130.6, 97.7), turned to -90 degrees

Commit message: update
Parts:
- K1, K2: footprint Semiconductor:DIP-10 -> Others:OMRON G6H-2-100
- moved LED1 61.1 mm to (104.6, 62.7)
- moved R4 49.0 mm to (118.4, 90.8), turned to 90 degrees
- moved R2 47.2 mm to (118.4, 74.5), turned to -90 degrees
- moved R1 46.4 mm to (120.8, 62.7), turned to 0 degrees
- moved R5 40.6 mm to (123.4, 90.2), turned to 90 degrees
- moved P1 27.7 mm to (108.1, 81.5)
- moved R3 27.2 mm to (123.2, 76.5), turned to -90 degrees
- moved K2 24.1 mm to (136.8, 90.9), turned to -90 degrees
- moved K1 21.7 mm to (136.8, 73.1), turned to -90 degrees
Connections:
- K1 pad 5: (no net) -> unconnected-(K1-Pad5)
- K1 pad 6: (no net) -> unconnected-(K1-Pad6)
- K2 pad 5: (no net) -> unconnected-(K2-Pad5)
- K2 pad 6: (no net) -> unconnected-(K2-Pad6)
Routing:
- net GND: track 0.00 -> 70.5 mm
- net /+24V: track 0.00 -> 69.7 mm
- net /+12V: track 0.00 -> 57.5 mm
- net Net-(K2-Pad4): track 0.00 -> 21.7 mm
- net Net-(K1-Pad4): track 0.00 -> 19.3 mm
- net /K2b: track 0.00 -> 18.4 mm
- net Net-(K2-Pad7): track 0.00 -> 16.6 mm
- net /K1b: track 0.00 -> 15.8 mm
- net Net-(K1-Pad7): track 0.00 -> 14.7 mm
- net Net-(LED1-Pad1): track 0.00 -> 12.8 mm
- net /K2a: track 0.00 -> 11.4 mm
- net /K1a: track 0.00 -> 10.3 mm
- net (no net): vias 0 -> 2
Other:
- board outline added: 70 x 40 mm
- board text added: "+12V"
- board text added: "+24V"
- board text added: "GND"
- board text added: "K1a"
- board text added: "K1b"
- board text added: "K2a"
- board text added: "K2b"
