File: MRLY220519.kicad_sch (KiCad schematic)
At the start: 2 parts

Commit message: updat
Parts:
- removed SW?: FUJITSU A-12W-K, symbol Switches:FUJITSU A-12W-K
- added SW? (x2): OMRON G6H-2-100, Passive:OMRON G6H-2-100, symbol Switches:OMRON G6H-2-100
Other:
- note added: "- DIP tok - Terminal block ellenoldal - 1K00 resistor - LED + resistor G6H-2-100"
- note added: "24V 42-17-17"
- note removed: "- DIP tok - Terminal block ellenoldal - 1K00 resistor - LED + resistor"
- note removed: "A-12 W-K A-12W-K 42-18-10"
Changed lines of the file:
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@@
 (kicad_sch (version 20211123) (generator eeschema)
   (paper "A4")
-  (text "A-12 W-K\n\nA-12W-K\n\n42-18-10" (at 191.77 30.48 0)
+  (text "\n24V\n\n42-17-17 \n" (at 185.42 30.48 0)
     (effects (font (size 1.27 1.27)) (justify left bottom))
   )
-  (text "- DIP tok\n- Terminal block ellenoldal\n- 1K00 resistor\n- LED + resistor"
-    (at 187.96 41.91 0)
+  (text "- DIP tok\n- Terminal block ellenoldal\n- 1K00 resistor\n- LED + resistor\n\nG6H-2-100"
+    (at 184.15 44.45 0)
     (effects (font (size 1.27 1.27)) (justify left bottom))
+  )
+  (symbol (lib_id "Switches:OMRON G6H-2-100") (at 194.31 74.93 0) (unit 1)
+    (in_bom yes) (on_board yes) (fields_autoplaced)
+    (property "Reference" "SW?" (id 0) (at 196.85 68.58 0))
+    (property "Value" "OMRON G6H-2-100" (id 1) (at 199.39 92.075 0)
+      (effects (font (size 1.27 1.27)) hide)
+    )
+    (property "Footprint" "Passive:OMRON G6H-2-100" (id 2) (at 194.31 67.31 0)
+      (effects (font (size 1.27 1.27)) hide)
+    )
+    (property "Datasheet" "${KNV_DATASHEET}\\AZ850.pdf" (id 3) (at 195.58 93.98 0)
+      (effects (font (size 1.27 1.27)) hide)
+    )
+    (property "Comment" "G6H-2-100" (id 4) (at 196.85 71.12 0))
+    (property "Manufacturer" "FUJITSU;ZETTLER" (id 5) (at 195.58 101.6 0)
+      (effects (font (size 1.27 1.27)) hide)
+    )
+    (property "ManufacturerPartNo" "A-24W-K;AZ850-24;" (id 6) (at 195.58 99.06 0)
+      (effects (font (size 1.27 1.27)) hide)
+    )
+    (property "Supplier" "TME-A-24W-K;TME-AZ850-24;" (id 7) (at 195.58 96.52 0)
+      (effects (font (size 1.27 1.27)) hide)
+    )
+    (pin "1")
+    (pin "10")
+    (pin "2")
+    (pin "3")
+    (pin "4")
+    (pin "7")
+    (pin "8")
+    (pin "9")
   )
   (symbol (lib_id "Connectors:Terminal Block 6 3.81 Straight") (at 236.22 60.96 0) (unit 1)
@@
     (pin "6")
   )
-  (symbol (lib_id "Switches:FUJITSU A-12W-K") (at 199.39 64.77 0) (unit 1)
+  (symbol (lib_id "Switches:OMRON G6H-2-100") (at 194.31 54.61 0) (unit 1)
     (in_bom yes) (on_board yes) (fields_autoplaced)
-    (property "Reference" "SW?" (id 0) (at 201.93 59.3303 0))
-    (property "Value" "FUJITSU A-12W-K" (id 1) (at 204.47 81.915 0)
+    (property "Reference" "SW?" (id 0) (at 196.85 48.26 0))
+    (property "Value" "OMRON G6H-2-100" (id 1) (at 199.39 71.755 0)
       (effects (font (size 1.27 1.27)) hide)
     )
-    (property "Footprint" "" (id 2) (at 199.39 57.15 0)
+    (property "Footprint" "Passive:OMRON G6H-2-100" (id 2) (at 194.31 46.99 0)
       (effects (font (size 1.27 1.27)) hide)
     )
-    (property "Datasheet" "${KNV_DATASHEET}\\5M.pdf" (id 3) (at 200.66 83.82 0)
+    (property "Datasheet" "${KNV_DATASHEET}\\AZ850.pdf" (id 3) (at 195.58 73.66 0)
       (effects (font (size 1.27 1.27)) hide)
     )
-    (property "Comment" "A-12W-K" (id 4) (at 201.93 62.1054 0))
-    (property "Manufacturer" "FUJITSU" (id 5) (at 200.66 91.44 0)
+    (property "Comment" "G6H-2-100" (id 4) (at 196.85 50.8 0))
+    (property "Manufacturer" "FUJITSU;ZETTLER" (id 5) (at 195.58 81.28 0)
       (effects (font (size 1.27 1.27)) hide)
     )
-    (property "ManufacturerPartNo" "A-12W-K;" (id 6) (at 200.66 88.9 0)
+    (property "ManufacturerPartNo" "A-24W-K;AZ850-24;" (id 6) (at 195.58 78.74 0)
       (effects (font (size 1.27 1.27)) hide)
     )
-    (property "Supplier" "TME-A-12W-K;" (id 7) (at 200.66 86.36 0)
+    (property "Supplier" "TME-A-24W-K;TME-AZ850-24;" (id 7) (at 195.58 76.2 0)
       (effects (font (size 1.27 1.27)) hide)
     )
@@
       (reference "P?") (unit 1) (value "Terminal Block 6 3.81 Straight") (footprint "")
     )
-    (path "/aec40859-dddb-4aa7-9566-0d4ab09d1189"
-      (reference "SW?") (unit 1) (value "FUJITSU A-12W-K") (footprint "")
+    (path "/5a83c478-c98d-4120-9ecb-99e35fd2c85e"
+      (reference "SW?") (unit 1) (value "OMRON G6H-2-100") (footprint "Passive:OMRON G6H-2-100")
+    )
+    (path "/c9e3168c-bc1d-46b9-a241-745d3c32565c"
+      (reference "SW?") (unit 1) (value "OMRON G6H-2-100") (footprint "Passive:OMRON G6H-2-100")
     )
   )

Commit message: update
Parts:
- removed P?: Terminal Block 6 3.81 Straight, symbol Connectors:Terminal Block 6 3.81 Straight
- removed SW? (x2): OMRON G6H-2-100, Passive:OMRON G6H-2-100, symbol Switches:OMRON G6H-2-100
- added K? (x2): OMRON G6H-2-100, Passive:OMRON G6H-2-100, symbol Switches:OMRON G6H-2-100
- added P?: Terminal Block 8 3.81 Straight, Connectors:Terminal Block 8 3.81 Straight, symbol Connectors:Terminal Block 8 3.81 Straight
- added R? (x4): Resistor 0207 1K00, Passive:R0207 Axial Horizontal, symbol Passive:Resistor 0207 1K00
Connections:
- new net: K?.1, K?.1
- new net: K?.3, K?.3, K?.8, K?.8
- new net: K?.4, R?.1 (x2)
- new net: K?.7, R?.1 (x2)
- new net GND: K?.10, K?.10
- new net K1a: P?.4, R?.2
- new net K1b: P?.5, R?.2
- new net K2a: P?.6, R?.2
- new net K2b: P?.7, R?.2
- no-connect marks 0 -> 4

Commit message: update
Parts:
- added LED1: 3mm Green, Passive:LED RAD GRE 3mm, symbol LED:3mm Green
- added R1: Resistor 0207 10K0, Passive:R0207 Axial Horizontal, symbol Passive:Resistor 0207 10K0
- K1, K2: renamed from K?; footprint Passive:OMRON G6H-2-100 -> Semiconductor:DIP-10
- P1: renamed from P?; footprint Connectors:Terminal Block 8 3.81 Straight -> Connectors:Terminal Block 1x08 P3.81 Straight
- R2, R3, R4, R5: renamed from R?; Manufacturer VIKING -> LSE; ManufacturerPartNo (none) -> 1K00 0.6W 1% MF0207;; Supplier (none) -> LOM-02-01-43;
Connections:
- net GND: now also P1.1 (Pin_a1), R1.2
- net +24V: now reaches K1.1, K2.1
- net +24V: now also P1.2, LED1.2 (A)
- net +12V: now reaches K1.3, K1.8, K2.3, K2.8
- net +12V: now also P1.8
- new net: LED1.1 (K), R1.1
- no-connect marks 4 -> 5
Other:
- note removed: "- DIP tok - Terminal block ellenoldal - 1K00 resistor - LED + resistor G6H-2-100"
- note removed: "24V 42-17-17"
- moved on the sheet: K1, K2, P1, R2, R3, R4, R5

Commit message: update
Parts:
- added S1, S2: DIP-14 Socket, symbol Accessories:DIP-14 Socket
- added W1: Terminal Block 01x08 P3.81 Plug, symbol ConnectorsOtherSide:Terminal Block 01x08 P3.81 Plug
- P1: footprint Connectors:Terminal Block 1x08 P3.81 Straight -> Connectors:Terminal Block 01x08 P3.81 Horizontal; symbol Connectors:Terminal Block 8 3.81 Straight -> Connectors:Terminal Block 01x08 P3.81 Horizontal; Comment MRT9P3.81/8 -> 15EDGRC3.81-08P; Manufacturer Stelvio -> DEGSON ELECTRONICS; ManufacturerPartNo MRT9P3.81/8; -> 15EDGRC3.81-08P;; Supplier LOM-43-19-25; TME-15EDGVC3.81-0P -> TME-15EDGRC3.81-08P
Changed lines of the file:
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@@
     (pin "2")
+  )
+  (symbol (lib_id "ConnectorsOtherSide:Terminal Block 01x08 P3.81 Plug") (at 171.45 96.52 0) (unit 1)
+    (in_bom yes) (on_board no) (fields_autoplaced)
+    (property "Reference" "W1" (id 0) (at 175.26 99.3774 0)
+      (effects (font (size 1.27 1.27)) (justify left))
+    )
+    (property "Value" "Terminal Block 01x08 P3.81 Plug" (id 1) (at 172.72 121.285 0)
+      (effects (font (size 1.27 1.27)) hide)
+    )
+    (property "Footprint" "" (id 2) (at 151.13 60.96 0)
+      (effects (font (size 1.27 1.27)) hide)
+    )
+    (property "Datasheet" "${KNV_DATASHEET}\\" (id 3) (at 172.72 109.855 0)
+      (effects (font (size 1.27 1.27)) hide)
+    )
+    (property "Comment" "15EDGK3.81-08P" (id 4) (at 175.26 101.9174 0)
+      (effects (font (size 1.27 1.27)) (justify left))
+    )
+    (property "Manufacturer" "DEGSON ELECTRONICS" (id 5) (at 172.085 125.73 0)
+      (effects (font (size 1.27 1.27)) hide)
+    )
+    (property "ManufacturerPartNo" "15EDGK3.81-08P;" (id 6) (at 173.99 112.395 0)
+      (effects (font (size 1.27 1.27)) hide)
+    )
+    (property "Supplier" "TME-15EDGK3.81-08P;" (id 7) (at 173.99 114.935 0)
+      (effects (font (size 1.27 1.27)) hide)
+    )
   )
   (symbol (lib_id "Switches:OMRON G6H-2-100") (at 115.57 105.41 0) (unit 1)
@@
     (pin "2")
   )
-  (symbol (lib_id "Connectors:Terminal Block 8 3.81 Straight") (at 158.75 90.17 0) (unit 1)
-    (in_bom yes) (on_board yes) (fields_autoplaced)
+  (symbol (lib_id "Connectors:Terminal Block 01x08 P3.81 Horizontal") (at 158.75 90.17 0) (unit 1)
+    (in_bom yes) (on_board yes)
     (property "Reference" "P1" (id 0) (at 162.56 99.0599 0)
       (effects (font (size 1.27 1.27)) (justify left))
@@
       (effects (font (size 1.27 1.27)) hide)
     )
-    (property "Footprint" "Connectors:Terminal Block 1x08 P3.81 Straight" (id 2) (at 138.43 54.61 0)
-      (effects (font (size 1.27 1.27)) hide)
-    )
-    (property "Datasheet" "${KNV_DATASHEET}\\" (id 3) (at 158.75 113.03 0)
-      (effects (font (size 1.27 1.27)) hide)
-    )
-    (property "Comment" "MRT9P3.81/8" (id 4) (at 162.56 101.5999 0)
-      (effects (font (size 1.27 1.27)) (justify left))
-    )
-    (property "Manufacturer" "Stelvio" (id 5) (at 173.99 124.46 0)
-      (effects (font (size 1.27 1.27)) hide)
-    )
-    (property "ManufacturerPartNo" "MRT9P3.81/8;" (id 6) (at 160.02 115.57 0)
-      (effects (font (size 1.27 1.27)) hide)
-    )
-    (property "Supplier" "LOM-43-19-25; TME-15EDGVC3.81-0P" (id 7) (at 160.02 118.11 0)
+    (property "Footprint" "Connectors:Terminal Block 01x08 P3.81 Horizontal" (id 2) (at 138.43 54.61 0)
+      (effects (font (size 1.27 1.27)) hide)
+    )
+    (property "Datasheet" "${KNV_DATASHEET}\\DEGSON 15EDGRC-3.81.pdf" (id 3) (at 158.75 113.03 0)
+      (effects (font (size 1.27 1.27)) hide)
+    )
+    (property "Comment" "15EDGRC3.81-08P" (id 4) (at 158.75 113.03 0))
+    (property "Manufacturer" "DEGSON ELECTRONICS" (id 5) (at 173.99 124.46 0)
+      (effects (font (size 1.27 1.27)) hide)
+    )
+    (property "ManufacturerPartNo" "15EDGRC3.81-08P;" (id 6) (at 160.02 115.57 0)
+      (effects (font (size 1.27 1.27)) hide)
+    )
+    (property "Supplier" "TME-15EDGRC3.81-08P" (id 7) (at 160.02 118.11 0)
       (effects (font (size 1.27 1.27)) hide)
     )
@@
     (pin "8")
   )
+  (symbol (lib_id "Accessories:DIP-14 Socket") (at 134.62 144.78 0) (unit 1)
+    (in_bom yes) (on_board no) (fields_autoplaced)
+    (property "Reference" "S2" (id 0) (at 140.97 141.3509 0)
+      (effects (font (size 1.27 1.27)) (justify left))
+    )
+    (property "Value" "DIP-14 Socket" (id 1) (at 137.16 154.686 0)
+      (effects (font (size 1.27 1.27)) hide)
+    )
+    (property "Footprint" "" (id 2) (at 134.747 152.146 0)
+      (effects (font (size 1.27 1.27)) hide)
+    )
+    (property "Datasheet" "" (id 3) (at 134.747 152.146 0)
+      (effects (font (size 1.27 1.27)) hide)
+    )
+    (property "Comment" "DIP-14 Socket" (id 4) (at 140.97 143.8909 0)
+      (effects (font (size 1.27 1.27)) (justify left))
+    )
+    (property "Manufacturer" "CONNFLY" (id 5) (at 133.985 141.605 0)
+      (effects (font (size 1.27 1.27)) hide)
+    )
+    (property "ManufacturerPartNo" "DS1001-01-14BT1NSF6X" (id 6) (at 135.255 139.7 0)
+      (effects (font (size 1.27 1.27)) hide)
+    )
+    (property "Supplier" "TME-GOLD-14P;" (id 7) (at 134.62 144.78 0)
+      (effects (font (size 1.27 1.27)) hide)
+    )
+  )
   (symbol (lib_id "Passive:Resistor 0207 10K0") (at 110.49 137.16 0) (unit 1)
     (in_bom yes) (on_board yes) (fields_autoplaced)
@@
     (pin "1")
     (pin "2")
+  )
+  (symbol (lib_id "Accessories:DIP-14 Socket") (at 134.62 134.62 0) (unit 1)
+    (in_bom yes) (on_board no) (fields_autoplaced)
+    (property "Reference" "S1" (id 0) (at 140.97 131.1909 0)
+      (effects (font (size 1.27 1.27)) (justify left))
+    )
+    (property "Value" "DIP-14 Socket" (id 1) (at 137.16 144.526 0)
+      (effects (font (size 1.27 1.27)) hide)
+    )
+    (property "Footprint" "" (id 2) (at 134.747 141.986 0)
+      (effects (font (size 1.27 1.27)) hide)
+    )
+    (property "Datasheet" "" (id 3) (at 134.747 141.986 0)
+      (effects (font (size 1.27 1.27)) hide)
+    )
+    (property "Comment" "DIP-14 Socket" (id 4) (at 140.97 133.7309 0)
+      (effects (font (size 1.27 1.27)) (justify left))
+    )
+    (property "Manufacturer" "CONNFLY" (id 5) (at 133.985 131.445 0)
+      (effects (font (size 1.27 1.27)) hide)
+    )
+    (property "ManufacturerPartNo" "DS1001-01-14BT1NSF6X" (id 6) (at 135.255 129.54 0)
+      (effects (font (size 1.27 1.27)) hide)
+    )
+    (property "Supplier" "TME-GOLD-14P;" (id 7) (at 134.62 134.62 0)
+      (effects (font (size 1.27 1.27)) hide)
+    )
   )
   (symbol (lib_id "CustomPowers:GND") (at 110.49 140.97 0) (unit 1)
@@
     )
     (path "/73a81f11-0a5e-4eab-b658-abc6825b92c4"
-      (reference "P1") (unit 1) (value "Terminal Block 8 3.81 Straight") (footprint "Connectors:Terminal Block 1x08 P3.81 Straight")
+      (reference "P1") (unit 1) (value "Terminal Block 8 3.81 Straight") (footprint "Connectors:Terminal Block 01x08 P3.81 Horizontal")
     )
     (path "/9759337a-e64f-4b6c-8775-f09221c04233"
@@
       (reference "R5") (unit 1) (value "Resistor 0207 1K00") (footprint "Passive:R0207 Axial Horizontal")
     )
-  )
+    (path "/a2cb6d3e-479e-42cb-b10e-9023dc32f8c9"
+      (reference "S1") (unit 1) (value "DIP-14 Socket") (footprint "")
+    )
+    (path "/7f732e05-2edb-4299-8934-f7b14de90012"
+      (reference "S2") (unit 1) (value "DIP-14 Socket") (footprint "")
+    )
+    (path "/159c7d91-abe4-4e62-9d3c-79a280f827b1"
+      (reference "W1") (unit 1) (value "Terminal Block 01x08 P3.81 Plug") (footprint "")
+    )
+  )

Commit message: update
Parts:
- K1, K2: footprint Semiconductor:DIP-10 -> Others:OMRON G6H-2-100
